File: pcb/DigitalYSplitter.brd (EAGLE design)
At the start: 40 x 30 mm, 42 parts, among them CN1 Battery, CON1 USB_MICROSMT+THRUHULE, CON2 M05X2NO_SILK, CON3 LED_OUT, CON5 LED_OUT, Q1 16MHz, SW1 BUTTON_1, SW2 BUTTON_2, U1 MK20D--VFM5, U3 74LVC1G17DCK, U4 74LVC1G17DCK, U5 74LVC1G17DCK, U6 TPD4S012, U7 74LVC1G17DCK

Commit message: Small corrections to the PCB
Parts:
- removed LED5: STATUS, adafruit:CHIPLED_0805
- removed R4: 470, adafruit:R0402
- moved LED1 14.8 mm to (16.4, -0.60), turned to 270 degrees
- renumbered LED6 to LED0
Connections:
- removed net N$16: LED1.A, R4.1
- removed net POWER_ENABLE: U1.29
- removed net STATUS: LED1.C, U1.31
- net +3V3: no longer R4.2
- net N$17: now also LED1.A; no longer LED5.A
- net TX: now also LED1.C; no longer LED5.C
Routing:
- net STATUS: track 24.7 -> 0.00 mm, vias 2 -> 0
- net +3V3: track 66.6 -> 54.8 mm
- net N$16: track 1.82 -> 0.00 mm
Changed lines of the file:
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@@
 <attribute name="VALUE" x="12.885" y="11.305" size="1.27" layer="27" rot="R180"/>
-</element>
-<element name="LED1" library="adafruit" package="CHIPLED_0805" value="STATUS" x="2.3" y="3.9" smashed="yes">
-<attribute name="NAME" x="1.08" y="3.98" size="1.016" layer="25" font="vector" rot="R90" align="center"/>
-<attribute name="VALUE" x="4.84" y="2.63" size="1.27" layer="27" rot="R90"/>
 </element>
 <element name="Q1" library="blinkinlabs" package="CRSYTAL_2520" value="16MHz" x="22.75" y="8.25" smashed="yes" rot="R180">
@@
 <attribute name="NAME" x="11.365" y="14.212" size="1.016" layer="25" font="vector" align="center"/>
 <attribute name="VALUE" x="9.065" y="12.218" size="1.27" layer="27"/>
-</element>
-<element name="R4" library="adafruit" package="R0402" value="470" x="3.95" y="3.9" smashed="yes" rot="R90">
-<attribute name="NAME" x="3.938" y="2.415" size="1.016" layer="25" font="vector" rot="R90" align="center"/>
-<attribute name="VALUE" x="5.982" y="3.265" size="1.27" layer="27" rot="R90"/>
 </element>
 <element name="CON1" library="blinkinlabs" package="USB_MICRO_THRUHOLE" value="USB_MICROSMT+THRUHULE" x="1.675" y="12.5" smashed="yes" rot="R270">
@@
 <element name="LED4" library="adafruit" package="CHIPLED_0805" value="STATUS" x="28.4" y="-0.6" rot="R270"/>
 <element name="R9" library="adafruit" package="R0402" value="470" x="16.4" y="-2.1"/>
-<element name="LED5" library="adafruit" package="CHIPLED_0805" value="STATUS" x="16.4" y="-0.6" rot="R270"/>
+<element name="LED1" library="adafruit" package="CHIPLED_0805" value="STATUS" x="16.4" y="-0.6" rot="R270"/>
 <element name="R10" library="adafruit" package="R0402" value="470" x="12.4" y="-2.1"/>
-<element name="LED6" library="adafruit" package="CHIPLED_0805" value="STATUS" x="12.4" y="-0.6" rot="R270"/>
+<element name="LED0" library="adafruit" package="CHIPLED_0805" value="STATUS" x="12.4" y="-0.6" rot="R270"/>
 </elements>
 <signals>
@@
 </signal>
 <signal name="+3V3">
-<contactref element="R4" pad="2"/>
 <contactref element="C2" pad="1"/>
 <contactref element="C1" pad="1"/>
@@
 <wire x1="17.5" y1="9.725" x2="17.5" y2="8.325" width="0.254" layer="1"/>
 <contactref element="CON2" pad="1"/>
-<wire x1="15.2" y1="2.84975" x2="15.2" y2="5.5" width="0.6096" layer="1"/>
-<wire x1="15.2" y1="5.5" x2="15.2" y2="8" width="0.6096" layer="1"/>
+<wire x1="15.2" y1="2.84975" x2="15.2" y2="8" width="0.6096" layer="1"/>
 <wire x1="15.2" y1="8" x2="15.2" y2="8.5" width="0.6096" layer="1"/>
 <wire x1="15.2" y1="8.5" x2="15.2" y2="8.6" width="0.6096" layer="1"/>
@@
 <wire x1="15.375" y1="11.125" x2="14.25" y2="10" width="0.6096" layer="16"/>
 <wire x1="14.25" y1="10" x2="13.8" y2="10" width="0.6096" layer="16"/>
-<wire x1="4.75" y1="5.5" x2="15.2" y2="5.5" width="0.254" layer="1"/>
-<wire x1="3.95" y1="4.55" x2="3.95" y2="4.7" width="0.254" layer="1"/>
-<wire x1="3.95" y1="4.7" x2="4.75" y2="5.5" width="0.254" layer="1"/>
 <wire x1="15.2" y1="8.6" x2="13.8" y2="10" width="0.6096" layer="1"/>
 <wire x1="15.225" y1="8.525" x2="15.2" y2="8.5" width="0.2032" layer="1"/>
@@
 <wire x1="18.5" y1="5.48" x2="19.21" y2="4.77" width="0.2032" layer="1"/>
 <contactref element="CON2" pad="4"/>
-<contactref element="LED6" pad="C"/>
+<contactref element="LED0" pad="C"/>
 <wire x1="13.45" y1="-0.6" x2="13.45" y2="-0.15" width="0.2032" layer="1"/>
 <wire x1="13.45" y1="-0.15" x2="14.5" y2="0.9" width="0.2032" layer="1"/>
@@
 <wire x1="19" y1="9.725" x2="19" y2="6.75" width="0.2032" layer="1"/>
 <contactref element="CON2" pad="5"/>
-<contactref element="LED5" pad="C"/>
+<contactref element="LED1" pad="C"/>
 <wire x1="17.45" y1="-0.6" x2="17.45" y2="0.05" width="0.2032" layer="1"/>
 <wire x1="17.45" y1="0.05" x2="17.8" y2="0.4" width="0.2032" layer="1"/>
@@
 <wire x1="17.6" y1="17.5" x2="18.5" y2="16.6" width="0.2032" layer="1"/>
 <wire x1="18.5" y1="16.6" x2="18.5" y2="15.275" width="0.2032" layer="1"/>
-</signal>
-<signal name="STATUS">
-<contactref element="LED1" pad="C"/>
-<wire x1="9" y1="7.5" x2="9.25" y2="7.75" width="0.2032" layer="1"/>
-<wire x1="9.25" y1="7.75" x2="9.25" y2="11.75" width="0.2032" layer="1"/>
-<contactref element="U1" pad="31"/>
-<wire x1="17" y1="15.275" x2="17" y2="16.25" width="0.2032" layer="1"/>
-<wire x1="17" y1="16.25" x2="16.75" y2="16.5" width="0.2032" layer="1"/>
-<via x="11.25" y="14.75" extent="1-16" drill="0.3"/>
-<via x="9.5" y="12" extent="1-16" drill="0.3"/>
-<wire x1="9" y1="7.5" x2="4.75" y2="7.5" width="0.2032" layer="1"/>
-<wire x1="4.75" y1="7.5" x2="4.5" y2="7.25" width="0.2032" layer="1"/>
-<wire x1="4.5" y1="7.25" x2="4.5" y2="6.25" width="0.2032" layer="1"/>
-<wire x1="4.5" y1="6.25" x2="4" y2="5.75" width="0.2032" layer="1"/>
-<wire x1="4" y1="5.75" x2="2.75" y2="5.75" width="0.2032" layer="1"/>
-<wire x1="2.75" y1="5.75" x2="2.3" y2="5.3" width="0.2032" layer="1"/>
-<wire x1="2.3" y1="4.95" x2="2.3" y2="5.3" width="0.2032" layer="1"/>
-<wire x1="9.25" y1="11.75" x2="9.5" y2="12" width="0.2032" layer="1"/>
-<wire x1="9.5" y1="12" x2="11" y2="13.5" width="0.2032" layer="16"/>
-<wire x1="12.25" y1="16.5" x2="16.75" y2="16.5" width="0.2032" layer="1"/>
-<wire x1="11.25" y1="14.75" x2="11.25" y2="15.5" width="0.2032" layer="1"/>
-<wire x1="11.25" y1="15.5" x2="12.25" y2="16.5" width="0.2032" layer="1"/>
-<wire x1="11" y1="13.5" x2="11" y2="14.5" width="0.2032" layer="16"/>
-<wire x1="11" y1="14.5" x2="11.25" y2="14.75" width="0.2032" layer="16"/>
-</signal>
-<signal name="N$16">
-<contactref element="R4" pad="1"/>
-<contactref element="LED1" pad="A"/>
-<wire x1="3.95" y1="3.25" x2="2.7" y2="3.25" width="0.254" layer="1"/>
-<wire x1="2.7" y1="3.25" x2="2.3" y2="2.85" width="0.254" layer="1"/>
 </signal>
 <signal name="RESET">
@@
 <wire x1="28.85" y1="16.1" x2="30.98" y2="18.23" width="0.2032" layer="1"/>
 <wire x1="30.98" y1="18.23" x2="31.246" y2="18.23" width="0.2032" layer="1"/>
-</signal>
-<signal name="POWER_ENABLE">
-<contactref element="U1" pad="29"/>
 </signal>
 <signal name="PA4">
@@
 <signal name="N$17">
 <contactref element="R9" pad="1"/>
-<contactref element="LED5" pad="A"/>
+<contactref element="LED1" pad="A"/>
 <wire x1="15.35" y1="-0.6" x2="15.35" y2="-1.7" width="0.2032" layer="1"/>
 <wire x1="15.35" y1="-1.7" x2="15.75" y2="-2.1" width="0.2032" layer="1"/>
@@
 <signal name="N$18">
 <contactref element="R10" pad="1"/>
-<contactref element="LED6" pad="A"/>
+<contactref element="LED0" pad="A"/>
 <wire x1="11.35" y1="-0.6" x2="11.35" y2="-1.7" width="0.2032" layer="1"/>
 <wire x1="11.35" y1="-1.7" x2="11.75" y2="-2.1" width="0.2032" layer="1"/>

Commit message: Small fixes to the PCB for clarity
Connections:
- net FLASH_MOSI renamed INPUT_MOSI
- new net INPUT_MISO: U1.28
- new net INPUT_SCK: U1.26
- net FLASH_MISO: no longer U1.28
- net FLASH_SCK: no longer U1.26
Routing:
- net FLASH_MISO: track 7.51 -> 6.19 mm
- net FLASH_SCK: track 4.82 -> 3.69 mm
Changed lines of the file:
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@@
 </signal>
 <signal name="FLASH_SCK">
-<contactref element="U1" pad="26"/>
 <contactref element="D3" pad="C"/>
 <contactref element="R5" pad="1"/>
 <wire x1="18.55" y1="18.1" x2="20.15" y2="18.1" width="0.2032" layer="1"/>
-<wire x1="19.5" y1="15.275" x2="19.5" y2="16.4" width="0.2032" layer="1"/>
 <wire x1="19.5" y1="16.4" x2="18.6" y2="17.3" width="0.2032" layer="1"/>
 <wire x1="18.6" y1="17.3" x2="18.6" y2="18.05" width="0.2032" layer="1"/>
 <wire x1="18.6" y1="18.05" x2="18.55" y2="18.1" width="0.2032" layer="1"/>
 </signal>
-<signal name="FLASH_MOSI">
+<signal name="INPUT_MOSI">
 <contactref element="U1" pad="27"/>
 </signal>
 <signal name="FLASH_MISO">
-<contactref element="U1" pad="28"/>
 <contactref element="D2" pad="C"/>
 <contactref element="R3" pad="1"/>
@@
 <wire x1="17.6" y1="19.8" x2="17.6" y2="17.5" width="0.2032" layer="1"/>
 <wire x1="17.6" y1="17.5" x2="18.5" y2="16.6" width="0.2032" layer="1"/>
-<wire x1="18.5" y1="16.6" x2="18.5" y2="15.275" width="0.2032" layer="1"/>
 </signal>
 <signal name="RESET">
@@
 <wire x1="11.35" y1="-1.7" x2="11.75" y2="-2.1" width="0.2032" layer="1"/>
 </signal>
+<signal name="INPUT_SCK">
+<contactref element="U1" pad="26"/>
+</signal>
+<signal name="INPUT_MISO">
+<contactref element="U1" pad="28"/>
+</signal>
 </signals>

Commit message: Schematic bugfix: can't use diodes for level shifting, they're too slow.
Parts:
- removed D2, D3: 3.3V, SparkFun-DiscreteSemi:SOD-323
- removed R3, R5: 470, adafruit:R0402
- added U2, U8: 74LVC1G17DCK, 74xx-little-us:SC70-5
Connections:
- removed net FLASH_MISO: D2.C, R3.1
- removed net FLASH_SCK: D3.C, R5.1
- net +3V3: now also U2.5, U8.5
- net GND: now also U2.3, U8.3; no longer D2.A, D3.A
- net INPUT_MISO: now also U2.4
- net INPUT_SCK: now also U8.4
- net N$6: now also U2.2; no longer R3.2
- net N$8: now also U8.2; no longer R5.2
Routing:
- net +3V3: track 54.8 -> 65.5 mm, vias 8 -> 9
- net FLASH_MISO: track 6.19 -> 0.00 mm
- net FLASH_SCK: track 3.69 -> 0.00 mm
- net INPUT_MISO: track 0.00 -> 3.35 mm
- net INPUT_SCK: track 0.00 -> 3.23 mm
- net N$8: track 5.37 -> 3.60 mm
- net GND: vias 40 -> 41
Changed lines of the file:
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@@
 <attribute name="VALUE" x="15.73" y="19.825" size="1.27" layer="27"/>
-</element>
-<element name="R3" library="adafruit" package="R0402" value="470" x="20.7" y="20.2" smashed="yes"/>
-<element name="R5" library="adafruit" package="R0402" value="470" x="20.8" y="18.1" smashed="yes"/>
-<element name="D2" library="SparkFun-DiscreteSemi" package="SOD-323" value="3.3V" x="17.4" y="20.2" smashed="yes" rot="R180">
-<attribute name="PROD_ID" value="DIO-11284" x="17.4" y="20.2" size="1.778" layer="27" rot="R180" display="off"/>
-</element>
-<element name="D3" library="SparkFun-DiscreteSemi" package="SOD-323" value="3.3V" x="17.4" y="18.1" smashed="yes" rot="R180">
-<attribute name="PROD_ID" value="DIO-11284" x="17.4" y="18.1" size="1.778" layer="27" rot="R180" display="off"/>
 </element>
 <element name="R6" library="adafruit" package="R0402" value="470" x="20.4" y="-2.1"/>
@@
 <element name="R10" library="adafruit" package="R0402" value="470" x="12.4" y="-2.1"/>
 <element name="LED0" library="adafruit" package="CHIPLED_0805" value="STATUS" x="12.4" y="-0.6" rot="R270"/>
+<element name="U2" library="74xx-little-us" package="SC70-5" value="74LVC1G17DCK" x="18" y="19" rot="R180"/>
+<element name="U8" library="74xx-little-us" package="SC70-5" value="74LVC1G17DCK" x="21" y="19" rot="R180"/>
 </elements>
 <signals>
@@
 <via x="24.35" y="17.4" extent="1-16" drill="0.3"/>
 <contactref element="JP1" pad="4"/>
-<contactref element="D3" pad="A"/>
-<contactref element="D2" pad="A"/>
 <via x="23.15" y="20.2" extent="1-16" drill="0.3"/>
 <via x="23.25" y="19.2" extent="1-16" drill="0.3"/>
+<contactref element="U2" pad="3"/>
+<contactref element="U8" pad="3"/>
+<via x="19.45" y="20.4" extent="1-16" drill="0.3"/>
 </signal>
 <signal name="N$2">
@@
 <wire x1="16.67" y1="2.23" x2="16.67" y2="-1.72" width="0.4064" layer="16"/>
 <wire x1="16.67" y1="-1.72" x2="17.05" y2="-2.1" width="0.4064" layer="16"/>
+<contactref element="U8" pad="5"/>
+<contactref element="U2" pad="5"/>
+<wire x1="21.65" y1="18.15" x2="21.65" y2="18.75" width="0.2032" layer="1"/>
+<wire x1="21.65" y1="18.75" x2="21.4" y2="19" width="0.2032" layer="1"/>
+<wire x1="21.4" y1="19" x2="18.65" y2="19" width="0.2032" layer="1"/>
+<wire x1="18.65" y1="19" x2="17.2" y2="19" width="0.2032" layer="1"/>
+<wire x1="17.2" y1="19" x2="15.4" y2="17.2" width="0.2032" layer="1"/>
+<via x="15.4" y="17.2" extent="1-16" drill="0.3"/>
+<wire x1="15.4" y1="17.2" x2="15.4" y2="15.15" width="0.2032" layer="16"/>
+<wire x1="15.4" y1="15.15" x2="15.375" y2="15.125" width="0.2032" layer="16"/>
+<wire x1="18.65" y1="18.15" x2="18.65" y2="19" width="0.2032" layer="1"/>
 </signal>
 <signal name="TCLK">
@@
 <wire x1="26.5" y1="10.5" x2="27.15" y2="10.5" width="0.2032" layer="1"/>
 </signal>
-<signal name="FLASH_SCK">
-<contactref element="D3" pad="C"/>
-<contactref element="R5" pad="1"/>
-<wire x1="18.55" y1="18.1" x2="20.15" y2="18.1" width="0.2032" layer="1"/>
-<wire x1="19.5" y1="16.4" x2="18.6" y2="17.3" width="0.2032" layer="1"/>
-<wire x1="18.6" y1="17.3" x2="18.6" y2="18.05" width="0.2032" layer="1"/>
-<wire x1="18.6" y1="18.05" x2="18.55" y2="18.1" width="0.2032" layer="1"/>
-</signal>
 <signal name="INPUT_MOSI">
 <contactref element="U1" pad="27"/>
-</signal>
-<signal name="FLASH_MISO">
-<contactref element="D2" pad="C"/>
-<contactref element="R3" pad="1"/>
-<wire x1="20.05" y1="20.2" x2="18.55" y2="20.2" width="0.2032" layer="1"/>
-<wire x1="18.55" y1="20.2" x2="18" y2="20.2" width="0.2032" layer="1"/>
-<wire x1="18" y1="20.2" x2="17.6" y2="19.8" width="0.2032" layer="1"/>
-<wire x1="17.6" y1="19.8" x2="17.6" y2="17.5" width="0.2032" layer="1"/>
-<wire x1="17.6" y1="17.5" x2="18.5" y2="16.6" width="0.2032" layer="1"/>
 </signal>
 <signal name="RESET">
@@
 <wire x1="6.5" y1="18.5" x2="5.85" y2="18.5" width="0.2032" layer="1"/>
 <contactref element="U1" pad="30"/>
-<wire x1="17.5" y1="15.275" x2="17.5" y2="16.496" width="0.2032" layer="1"/>
-<wire x1="17.5" y1="16.496" x2="16.996" y2="17" width="0.2032" layer="1"/>
-<wire x1="16.996" y1="17" x2="14.25" y2="17" width="0.2032" layer="1"/>
-<wire x1="14.25" y1="17" x2="13.65" y2="17.6" width="0.2032" layer="1"/>
-<wire x1="13.65" y1="17.6" x2="13.65" y2="18.5" width="0.2032" layer="1"/>
+<wire x1="17.5" y1="15.275" x2="17.5" y2="15.996" width="0.2032" layer="1"/>
+<wire x1="17.5" y1="15.996" x2="16.996" y2="16.5" width="0.2032" layer="1"/>
+<wire x1="16.996" y1="16.5" x2="14.25" y2="16.5" width="0.2032" layer="1"/>
+<wire x1="14.25" y1="16.5" x2="13.65" y2="17.1" width="0.2032" layer="1"/>
+<wire x1="13.65" y1="17.1" x2="13.65" y2="18.5" width="0.2032" layer="1"/>
 </signal>
 <signal name="LED_DATA1">
@@
 <signal name="N$6">
 <contactref element="JP1" pad="2"/>
-<contactref element="R3" pad="2"/>
-<wire x1="19.54" y1="23" x2="19.54" y2="22.76" width="0.2032" layer="1"/>
-<wire x1="19.54" y1="22.76" x2="21.25" y2="21.05" width="0.2032" layer="1"/>
-<wire x1="21.25" y1="21.05" x2="21.3" y2="21" width="0.2032" layer="1"/>
-<wire x1="21.35" y1="20.2" x2="21.35" y2="20.95" width="0.2032" layer="1"/>
-<wire x1="21.35" y1="20.95" x2="21.3" y2="21" width="0.2032" layer="1"/>
+<wire x1="19.54" y1="23" x2="19.54" y2="22.54" width="0.2032" layer="1"/>
+<contactref element="U2" pad="2"/>
+<wire x1="19.54" y1="22.54" x2="18" y2="21" width="0.2032" layer="1"/>
+<wire x1="18" y1="21" x2="18" y2="19.85" width="0.2032" layer="1"/>
 </signal>
 <signal name="N$8">
 <contactref element="JP1" pad="3"/>
-<contactref element="R5" pad="2"/>
-<wire x1="22.08" y1="23" x2="22.08" y2="18.38" width="0.2032" layer="1"/>
-<wire x1="21.45" y1="18.1" x2="21.8" y2="18.1" width="0.2032" layer="1"/>
-<wire x1="21.8" y1="18.1" x2="22.08" y2="18.38" width="0.2032" layer="1"/>
+<contactref element="U8" pad="2"/>
+<wire x1="22.08" y1="23" x2="22.08" y2="22.08" width="0.2032" layer="1"/>
+<wire x1="22.08" y1="22.08" x2="21" y2="21" width="0.2032" layer="1"/>
+<wire x1="21" y1="21" x2="21" y2="19.85" width="0.2032" layer="1"/>
 </signal>
 <signal name="N$13">
@@
 <signal name="INPUT_SCK">
 <contactref element="U1" pad="26"/>
+<contactref element="U8" pad="4"/>
+<wire x1="19.5" y1="15.275" x2="19.5" y2="16.5" width="0.2032" layer="1"/>
+<wire x1="19.5" y1="16.5" x2="20.35" y2="17.35" width="0.2032" layer="1"/>
+<wire x1="20.35" y1="18.15" x2="20.35" y2="17.35" width="0.2032" layer="1"/>
 </signal>
 <signal name="INPUT_MISO">
 <contactref element="U1" pad="28"/>
+<contactref element="U2" pad="4"/>
+<wire x1="17.35" y1="18.15" x2="17.35" y2="17.65" width="0.2032" layer="1"/>
+<wire x1="17.35" y1="17.65" x2="18.5" y2="16.5" width="0.2032" layer="1"/>
+<wire x1="18.5" y1="16.5" x2="18.5" y2="15.275" width="0.2032" layer="1"/>
 </signal>
 </signals>
